Commit message: ⚡️ add : Inertial parameters and calculations for the caster wheel

File: lmr1_description/urdf/common/inertials.xacro (robot description, xacro)
@@ -13,4 +13,17 @@
             iyz="0.0"
             izz="${(1.0/12.0) * mass * (length*length + width*width)}"/>
+    </xacro:macro>
+    <!-- =============================================== -->
+    <!-- Solid Sphere Inertia -->
+    <!-- =============================================== -->
+    <xacro:macro name="sphere_inertia"
+                 params="mass radius">
+        <inertia
+            ixx="${(2.0/5.0) * mass * radius * radius}"
+            ixy="0.0"
+            ixz="0.0"
+            iyy="${(2.0/5.0) * mass * radius * radius}"
+            iyz="0.0"
+            izz="${(2.0/5.0) * mass * radius * radius}" />
     </xacro:macro>
     <!-- ========================================= -->

File: lmr1_description/urdf/components/caster.xacro (robot description, xacro)
@@ -2,4 +2,11 @@
 <robot xmlns:xacro="http://www.ros.org/wiki/xacro">
     <link name="caster_wheel_link">
+        <inertial>
+            <origin xyz="0 0 0" rpy="0 0 0"/>
+            <mass value="${caster_mass}"/>
+            <xacro:sphere_inertia
+                mass="${caster_mass}"
+                radius="${caster_radius}"/>
+        </inertial>
         <!-- collision -->
         <collision>
