Commit message: 🔧 edit : Modification of robot parameters in properties.xacro
- wheel mass
- caster mass and radius

File: lmr1_description/urdf/common/properties.xacro (robot description, xacro)
@@ -14,7 +14,7 @@
     <xacro:property name="base_mass" value="2.0"/>
     <!-- base visual/collision offset -->
-    <xacro:property name="base_offset_x" value="0.0"/>
+    <xacro:property name="base_offset_x" value="0.065"/>
     <xacro:property name="base_offset_y" value="0.0"/>
-    <xacro:property name="base_offset_z" value="0.0"/>
+    <xacro:property name="base_offset_z" value="0.055"/>
     <!-- ==================== -->
     <!-- Wheel Dimensions -->
@@ -22,5 +22,5 @@
     <xacro:property name="wheel_radius" value="0.0325"/>
     <xacro:property name="wheel_width"  value="0.020"/>
-    <xacro:property name="wheel_mass" value="0.05"/>
+    <xacro:property name="wheel_mass" value="0.150"/>
     <!-- wheel locations -->
     <xacro:property name="wheel_offset_x" value="0.0"/>
@@ -30,5 +30,6 @@
     <!-- Caster -->
     <!-- ==================== -->
-    <xacro:property name="caster_radius" value="0.0075"/>
+    <xacro:property name="caster_radius" value="0.008"/>
+    <xacro:property name="caster_mass" value="0.05"/>
     <xacro:property name="caster_offset_x" value="0.175"/>
     <xacro:property name="caster_offset_y" value="0.0"/>

Commit message: 🔧 config : edit base link collision parameters

File: lmr1_description/urdf/common/properties.xacro (robot description, xacro)
@@ -11,5 +11,5 @@
     <xacro:property name="base_length" value="0.30"/>
     <xacro:property name="base_width"  value="0.18"/>
-    <xacro:property name="base_height" value="0.13"/>
+    <xacro:property name="base_height" value="0.10"/>
     <xacro:property name="base_mass" value="2.0"/>
     <!-- base visual/collision offset -->
