Commit message: ✨ feat : added IMU gazebo plugins and collision and inertial parameters

File: lmr1_description/urdf/components/sensors.xacro (robot description, xacro)
@@ -4,5 +4,22 @@
     <!-- IMU -->
     <!-- ======================== -->
-    <link name="imu_link"/>
+    <link name="imu_link">
+        <collision>
+            <geometry>
+                <box size="0.01 0.01 0.01"/>
+            </geometry>
+        </collision>
+        <inertial>
+            <origin xyz="0 0 0" rpy="0 0 0"/>
+            <mass value="0.01"/>
+            <inertia
+                ixx="0.000001"
+                ixy="0.0"
+                ixz="0.0"
+                iyy="0.000001"
+                iyz="0.0"
+                izz="0.000001"/>
+        </inertial>
+    </link>
     <joint name="imu_joint"
            type="fixed">

File: lmr1_description/urdf/robot.urdf.xacro (robot description, xacro)
@@ -71,8 +71,57 @@
     </gazebo>
     <gazebo reference="caster_wheel_link">
-        <mu1>0.5</mu1>
-        <mu2>0.5</mu2>
+        <mu1>0.6</mu1>
+        <mu2>0.6</mu2>
         <kp>100000.0</kp>
         <kd>10.0</kd>
     </gazebo>
+    <gazebo reference="lidar_link">
+        <sensor type="ray" name="ld19_lidar">
+            <pose>0 0 0 0 0 0</pose>
+            <visualize>false</visualize>
+            <update_rate>10</update_rate>
+            <ray>
+                <scan>
+                    <horizontal>
+                        <samples>450</samples>
+                        <resolution>1</resolution>
+                        <min_angle>-3.141592</min_angle>
+                        <max_angle>3.141592</max_angle>
+                    </horizontal>
+                </scan>
+                <range>
+                    <min>0.2</min>
+                    <max>12.0</max>
+                    <resolution>0.01</resolution>
+                </range>
+                <noise>
+                    <type>gaussian</type>
+                    <mean>0.0</mean>
+                    <stddev>0.01</stddev>
+                </noise>
+            </ray>
+            <plugin name="gazebo_ros_laser"
+                    filename="libgazebo_ros_laser.so">
+                <topicName>/scan</topicName>
+                <frameName>lidar_link</frameName>
+            </plugin>
+        </sensor>
+    </gazebo>
+  <gazebo reference="imu_link">
+        <gravity>true</gravity>
+        <sensor name="imu_sensor" type="imu">
+            <pose>0 0 0 0 0 0</pose>
+            <always_on>true</always_on>
+            <visualize>false</visualize>
+            <update_rate>100</update_rate>
+            <plugin filename="libgazebo_ros_imu_sensor.so" name="imu_plugin">
+                <topicName>imu</topicName>
+                <bodyName>imu_link</bodyName>
+                <updateRateHZ>100.0</updateRateHZ>
+                <gaussianNoise>0.002</gaussianNoise>
+                <frameName>imu_link</frameName>
+                <initialOrientationAsReference>false</initialOrientationAsReference>
+            </plugin>
+        </sensor>
+  </gazebo>
 </robot>
