Commit message: 🐛 fix : updated latest light weight meshes in URDF

File: lmr1_description/urdf/components/base.xacro (robot description, xacro)
@@ -23,5 +23,5 @@
                 rpy="0 0 0"/>
             <geometry>
-                <mesh filename="package://lmr1_description/meshes/base.dae"/>
+                <mesh filename="package://lmr1_description/meshes/base_light.dae"/>
             </geometry>
         </visual>

File: lmr1_description/urdf/robot.urdf (robot description, URDF)
Before this commit: robot lmr1, 6 links, 5 joints
Links:
- link base_link: geometry collision box size=0.3 0.18 0.1; visual mesh filename=package://lmr1_description/meshes/base_light.dae
- link caster_wheel_link: mass None -> 0.05; geometry collision sphere radius=0.008
- link imu_link: mass None -> 0.01; geometry collision box size=0.01 0.01 0.01
- link left_wheel_link: mass 0.05 -> 0.15; geometry collision cylinder length=0.02 radius=0.0325; visual mesh filename=package://lmr1_description/meshes/wheel_light.dae
- link right_wheel_link: mass 0.05 -> 0.15; geometry collision cylinder length=0.02 radius=0.0325; visual mesh filename=package://lmr1_description/meshes/wheel_light.dae

File: lmr1_description/urdf/robot.urdf.xacro (robot description, xacro)
@@ -16,5 +16,5 @@
         xyz="0 ${wheel_offset_y} ${wheel_offset_z}"
         rpy="-${PI/2} 0 0"
-        mesh_file="package://lmr1_description/meshes/wheel.dae"
+        mesh_file="package://lmr1_description/meshes/wheel_light.dae"
         axis="0 0 1"/>
     <!-- right wheel -->
@@ -24,5 +24,5 @@
         xyz="0 -${wheel_offset_y} ${wheel_offset_z}"
         rpy="${PI/2} 0 0"
-        mesh_file="package://lmr1_description/meshes/wheel.dae"
+        mesh_file="package://lmr1_description/meshes/wheel_light.dae"
         axis="0 0 -1"/>
     <gazebo>
