Commit message: 🔥 edit : reduced file volumes for better deployment

File: lmr1_description/web_viewer/public/robot/robot.urdf (robot description, URDF)
Before this commit: robot lmr1_web, 3 links, 2 joints
Links:
- link base_link: geometry visual mesh filename=./meshes/base.glb

Commit message: 🔥 edit : reduced file volumes for better deployment

File: lmr1_description/web_viewer/public/robot/robot.urdf (robot description, URDF)
Before this commit: robot lmr1_web, 3 links, 2 joints
Links:
- link base_link: geometry visual mesh filename=./meshes/base_light.dae

Commit message: 🎨 edit : reduced file volumes for better deployment

File: lmr1_description/web_viewer/public/robot/robot.urdf (robot description, URDF)
Before this commit: robot lmr1_web, 3 links, 2 joints
Links:
- link left_wheel_link: geometry visual mesh filename=./meshes/wheel_light.dae
- link right_wheel_link: geometry visual mesh filename=./meshes/wheel_light.dae
